File: cad/chickenguard/chickenguard.sch (KiCad schematic (older format))
At the start: 5 parts, among them J1 Conn_01x18, J2 Conn_01x18, J3 Screw_Terminal_01x16, J4 Screw_Terminal_01x12, J5 Jack-DC

Commit message: Schematic review.
Parts:
- added J6: Conn_01x04, symbol Connector_Generic:Conn_01x04
- added J7: Conn_01x02, symbol Connector_Generic:Conn_01x02
- added J8: Conn_01x03, symbol Connector_Generic:Conn_01x03
- J3: value Screw_Terminal_01x16 -> Screw Terminal
- J4: value Screw_Terminal_01x12 -> Screw Terminal
Connections:
- net labels added: 3V3, DCF77
- wire segments 74 -> 83
Other:
- note added: "10 M1DIR"
- note added: "21"
- note added: "36"
- note added: "7 MW2PWM"
- note added: "8 M2DIR"
- note added: "9 M1PWM"
- note added: "AVIN"
- note added: "GND"
- note added: "Motor Driver DRV8835"
- note added: "VCC"
- note added: "WARNING: Pins are mirrored!"
