File: cad/schematic/chickenguard.sch (KiCad schematic (older format))
At the start: 8 parts, among them J1 Conn_01x18, J2 Conn_01x18, J3 Screw Terminal, J4 Screw Terminal, J5 Jack-DC, J6 Conn_01x04, J7 Conn_01x02, J8 Conn_01x03

Commit message: css test.
Parts:
- added JP1, JP2, JP3, JP4, JP5, JP? (x2): Jumper_NO_Small, symbol Device:Jumper_NO_Small
- added RN1: 10K, Resistor_THT:R_Array_SIP9, symbol Device:R_Network08
Connections:
- net labels added: DECHO_BSWITCH, DTRIG_TSWITCH
- net labels removed: 3V3, DIST_ECHO, DIST_TRIGGER
- wire segments 83 -> 107
Other:
- note added: "7 M1DIR"
- note removed: "10 M1DIR"
- note removed: "7 MW2PWM"
- note removed: "8 M2DIR"
Changed lines of the file:
@@
 Text Notes 4650 3350 0    50   ~ 0
 GPIO21 SDA
-Text Label 2850 2450 0    50   ~ 0
-MOT_DRV
-Text Label 2850 2550 0    50   ~ 0
-MOT_DIR
-Text Label 2850 2350 0    50   ~ 0
-MOT_PWM
-Text Label 2850 2050 0    50   ~ 0
-DIST_TRIGGER
-Text Label 2850 2250 0    50   ~ 0
-DIST_ECHO
 Text Label 5600 2850 0    50   ~ 0
 UP_BUTTON
@@
 Wire Wire Line
 	8950 2050 8950 1700
-Text Label 2850 2850 0    50   ~ 0
-LUMINANCE
 $Comp
 L Connector:Screw_Terminal_01x16 J3
@@
 	5450 2750 6650 2750
 Wire Wire Line
-	6650 2450 6650 2550
-Wire Wire Line
-	6650 2550 6850 2550
-Wire Wire Line
-	5450 2450 6650 2450
-Wire Wire Line
 	6750 1650 6750 1750
 Wire Wire Line
@@
 	6750 1750 6750 1850
 Wire Wire Line
-	6650 1750 6650 1950
-Wire Wire Line
-	6650 1950 6750 1950
-Wire Wire Line
 	5450 1750 6650 1750
-Wire Wire Line
-	6750 1950 6750 2050
-Wire Wire Line
-	6750 2150 6850 2150
-Connection ~ 6750 1950
-Wire Wire Line
-	6750 1950 6850 1950
-Wire Wire Line
-	6850 2050 6750 2050
-Connection ~ 6750 2050
-Wire Wire Line
-	6750 2050 6750 2150
 Wire Notes Line
 	5500 3500 5500 1350
@@
 	1    0    0    -1
 $EndComp
-Text Label 5550 5050 0    50   ~ 0
-3V3
 Wire Wire Line
 	5350 4950 5750 4950
 Text Label 5550 4950 0    50   ~ 0
 GND
-Text Notes 4000 5200 0    50   ~ 0
-10 M1DIR
 Text Notes 4000 5100 0    50   ~ 0
 9 M1PWM
-Text Notes 4000 5000 0    50   ~ 0
-8 M2DIR
 Text Notes 4000 4850 0    50   ~ 0
-7 MW2PWM
+7 M1DIR
 Text Notes 4800 5050 0    50   ~ 0
 VCC
@@
 	3550 4600 5500 4600
 Wire Wire Line
-	2600 2550 2600 5200
-Wire Wire Line
-	3700 5200 2600 5200
+	2600 2550 2600 4850
 Wire Wire Line
 	2400 2350 2400 5100
@@
 Wire Wire Line
 	1750 3050 2700 3050
-Text Label 2850 2950 0    50   ~ 0
-DCF77
 Wire Wire Line
 	3600 2950 2800 2950
@@
 Wire Wire Line
 	1750 3150 2800 3150
+Wire Wire Line
+	3700 4850 2600 4850
+$Comp
+L Device:R_Network08 RN1
+U 1 1 5C86D958
+P 9400 3100
+F 0 "RN1" H 9780 3146 50  0000 L CNN
+F 1 "10K" H 9780 3055 50  0000 L CNN
+F 2 "Resistor_THT:R_Array_SIP9" V 9875 3100 50  0001 C CNN
+F 3 "http://www.vishay.com/docs/31509/csc.pdf" H 9400 3100 50  0001 C CNN
+	1    9400 3100
+	1    0    0    -1
+$EndComp
+$Comp
+L power:+5V #PWR01
+U 1 1 5C86D9D9
+P 9000 2800
+F 0 "#PWR01" H 9000 2650 50  0001 C CNN
+F 1 "+5V" H 9015 2973 50  0000 C CNN
+F 2 "" H 9000 2800 50  0001 C CNN
+F 3 "" H 9000 2800 50  0001 C CNN
+	1    9000 2800
+	1    0    0    -1
+$EndComp
+Wire Wire Line
+	9000 2900 9000 2800
+$Comp
+L Device:Jumper_NO_Small JP1
+U 1 1 5C86FC67
+P 9000 3500
+F 0 "JP1" V 9000 3453 50  0001 R CNN
+F 1 "Jumper_NO_Small" V 9045 3452 50  0001 R CNN
+F 2 "" H 9000 3500 50  0001 C CNN
+F 3 "~" H 9000 3500 50  0001 C CNN
+	1    9000 3500
+	0    1    1    0
+$EndComp
+$Comp
+L Device:Jumper_NO_Small JP2
+U 1 1 5C86FD2A
+P 9100 3500
+F 0 "JP2" V 9100 3548 50  0001 L CNN
+F 1 "Jumper_NO_Small" V 9145 3548 50  0001 L CNN
+F 2 "" H 9100 3500 50  0001 C CNN
+F 3 "~" H 9100 3500 50  0001 C CNN
+	1    9100 3500
+	0    1    1    0
+$EndComp
+$Comp
+L Device:Jumper_NO_Small JP3
+U 1 1 5C86FD50
+P 9200 3500
+F 0 "JP3" V 9200 3548 50  0001 L CNN
+F 1 "Jumper_NO_Small" V 9245 3548 50  0001 L CNN
+F 2 "" H 9200 3500 50  0001 C CNN
+F 3 "~" H 9200 3500 50  0001 C CNN
+	1    9200 3500
+	0    1    1    0
+$EndComp
+$Comp
+L Device:Jumper_NO_Small JP4
+U 1 1 5C86FD78
+P 9300 3500
+F 0 "JP4" V 9300 3548 50  0001 L CNN
+F 1 "Jumper_NO_Small" V 9345 3548 50  0001 L CNN
+F 2 "" H 9300 3500 50  0001 C CNN
+F 3 "~" H 9300 3500 50  0001 C CNN
+	1    9300 3500
+	0    1    1    0
+$EndComp
+$Comp
+L Device:Jumper_NO_Small JP5
+U 1 1 5C86FDA4
+P 9400 3500
+F 0 "JP5" V 9400 3548 50  0001 L CNN
+F 1 "Jumper_NO_Small" V 9445 3548 50  0001 L CNN
+F 2 "" H 9400 3500 50  0001 C CNN
+F 3 "~" H 9400 3500 50  0001 C CNN
+	1    9400 3500
+	0    1    1    0
+$EndComp
+Wire Wire Line
+	9000 3300 9000 3400
+Wire Wire Line
+	9100 3300 9100 3400
+Wire Wire Line
+	9200 3300 9200 3400
+Wire Wire Line
+	9300 3300 9300 3400
+Wire Wire Line
+	9400 3300 9400 3400
+Wire Wire Line
+	9000 3600 9000 3700
+Wire Wire Line
+	9000 3700 8350 3700
+Wire Wire Line
+	9100 3600 9100 3800
+Wire Wire Line
+	9100 3800 8350 3800
+Wire Wire Line
+	9200 3600 9200 3900
+Wire Wire Line
+	9200 3900 8350 3900
+Wire Wire Line
+	9300 3600 9300 4000
+Wire Wire Line
+	9300 4000 8350 4000
+Wire Wire Line
+	9400 3600 9400 4100
+Wire Wire Line
+	9400 4100 8350 4100
+Text Label 8350 3700 0    50   ~ 0
+DTRIG_TSWITCH
+Text Label 2850 2050 0    50   ~ 0
+DTRIG_TSWITCH
+Text Label 2850 2250 0    50   ~ 0
+DECHO_BSWITCH
+Text Label 2850 2350 0    50   ~ 0
+MOT_PWM
+Text Label 2850 2450 0    50   ~ 0
+MOT_DRV
+Text Label 2850 2550 0    50   ~ 0
+MOT_DIR
+Text Label 2850 2850 0    50   ~ 0
+LUMINANCE
+Text Label 2850 2950 0    50   ~ 0
+DCF77
+Text Label 8350 3800 0    50   ~ 0
+DECHO_BSWITCH
+Text Label 8350 3900 0    50   ~ 0
+STOP_SWITCH
+Text Label 8350 4000 0    50   ~ 0
+DOWN_BUTTON
+Text Label 8350 4100 0    50   ~ 0
+UP_BUTTON
+$Comp
+L Device:Jumper_NO_Small JP?
+U 1 1 5C89459F
+P 9500 3500
+F 0 "JP?" V 9500 3548 50  0001 L CNN
+F 1 "Jumper_NO_Small" V 9545 3548 50  0001 L CNN
+F 2 "" H 9500 3500 50  0001 C CNN
+F 3 "~" H 9500 3500 50  0001 C CNN
+	1    9500 3500
+	0    1    1    0
+$EndComp
+$Comp
+L Device:Jumper_NO_Small JP?
+U 1 1 5C8945BC
+P 9600 3500
+F 0 "JP?" V 9600 3548 50  0001 L CNN
+F 1 "Jumper_NO_Small" V 9645 3548 50  0001 L CNN
+F 2 "" H 9600 3500 50  0001 C CNN
+F 3 "~" H 9600 3500 50  0001 C CNN
+	1    9600 3500
+	0    1    1    0
+$EndComp
+Wire Wire Line
+	9500 3300 9500 3400
+Wire Wire Line
+	9600 3300 9600 3400
+Wire Wire Line
+	9500 3600 9500 4200
+Wire Wire Line
+	9500 4200 8350 4200
+Wire Wire Line
+	9600 3600 9600 4300
+Wire Wire Line
+	9600 4300 8350 4300
+Wire Wire Line
+	9700 3300 9700 4400
+Wire Wire Line
+	9700 4400 8350 4400
+Text Label 8350 4400 0    50   ~ 0
+DCF77
+Wire Wire Line
+	6750 1850 6750 1950
+Wire Wire Line
+	6750 1950 6850 1950
+Connection ~ 6750 1850
+Wire Wire Line
+	6850 2050 6750 2050
+Wire Wire Line
+	6650 1750 6650 2050
+Wire Wire Line
+	6750 2050 6750 2150
+Wire Wire Line
+	6750 2150 6850 2150
+Connection ~ 6750 2050
+Wire Wire Line
+	6750 2050 6650 2050
+Wire Wire Line
+	6750 2150 6750 2250
+Wire Wire Line
+	6750 2250 6850 2250
+Connection ~ 6750 2150
+Wire Wire Line
+	5450 2450 6850 2450
 $EndSCHEMATC

Commit message: errors fixed.
Connections:
- net labels added: BOTTOM_SWITCH, STOP_BUTTON, TOP_SWITCH
- wire segments 107 -> 113
Changed lines of the file:
@@
 Text Label 2850 1950 0    50   ~ 0
 RESET
-Text Label 5600 2450 0    50   ~ 0
-STOP_SWITCH
 $Comp
 L Connector:Jack-DC J5
@@
 $EndComp
 Wire Wire Line
-	3600 2550 2600 2550
-Wire Wire Line
-	2500 2450 3600 2450
+	3600 2550 2650 2550
 Wire Wire Line
-	2400 2350 3600 2350
+	2550 2450 3600 2450
 Wire Wire Line
-	2300 2250 3600 2250
+	2450 2350 3600 2350
 Wire Wire Line
-	2200 2050 3600 2050
+	2350 2250 3600 2250
 Wire Wire Line
 	1750 1950 1850 1950
@@
 	5450 1650 6750 1650
 Wire Wire Line
-	6750 2850 6750 2750
+	6650 2850 6650 2650
 Wire Wire Line
-	6750 2750 6850 2750
+	6650 2650 6850 2650
 Wire Wire Line
-	5450 2850 6750 2850
+	5450 2850 6650 2850
 Wire Wire Line
-	6650 2750 6650 2650
+	6550 2750 6550 2550
 Wire Wire Line
-	6650 2650 6850 2650
+	6550 2550 6850 2550
 Wire Wire Line
-	5450 2750 6650 2750
+	5450 2750 6550 2750
 Wire Wire Line
 	6750 1650 6750 1750
@@
 	3550 4600 5500 4600
 Wire Wire Line
-	2600 2550 2600 4850
+	2650 2550 2650 4850
 Wire Wire Line
-	2400 2350 2400 5100
+	2450 2350 2450 5100
 Wire Wire Line
-	2400 5100 3700 5100
+	2450 5100 3700 5100
 Wire Wire Line
-	2500 2450 2500 4250
+	2550 2450 2550 4250
 Wire Wire Line
-	2500 4250 5950 4250
+	2550 4250 5950 4250
 Wire Wire Line
 	5950 4250 5950 5050
@@
 GPIO34* ADC1_6
 Wire Wire Line
-	1750 2850 2200 2850
+	1750 2850 2250 2850
 Wire Wire Line
-	2200 2050 2200 2850
+	1750 2950 2350 2950
 Wire Wire Line
-	1750 2950 2300 2950
-Wire Wire Line
-	2300 2250 2300 2950
+	2350 2250 2350 2950
 Wire Wire Line
 	1750 3050 2700 3050
@@
 	1750 3150 2800 3150
 Wire Wire Line
-	3700 4850 2600 4850
+	3700 4850 2650 4850
 $Comp
 L Device:R_Network08 RN1
@@
 DTRIG_TSWITCH
 Text Label 2850 2050 0    50   ~ 0
-DTRIG_TSWITCH
+TOP_SWITCH
 Text Label 2850 2250 0    50   ~ 0
-DECHO_BSWITCH
+BOTTOM_SWITCH
 Text Label 2850 2350 0    50   ~ 0
 MOT_PWM
@@
 Connection ~ 6750 2150
 Wire Wire Line
-	5450 2450 6850 2450
+	3600 2050 2250 2050
+Wire Wire Line
+	2250 2050 2250 2850
+Wire Wire Line
+	3600 3050 2950 3050
+Text Label 2950 3050 0    50   ~ 0
+STOP_BUTTON
+Wire Wire Line
+	6850 2750 6750 2750
+Wire Wire Line
+	6750 2750 6750 2950
+Wire Wire Line
+	6750 2950 5950 2950
+Wire Wire Line
+	5950 2950 5950 4150
+Wire Wire Line
+	5950 4150 2950 4150
+Wire Wire Line
+	2950 4150 2950 3050
 $EndSCHEMATC

Commit message: Schematic review.
Connections:
- wire segments 113 -> 118
Changed lines of the file:
@@
 	2250 2050 2250 2850
 Wire Wire Line
-	3600 3050 2950 3050
-Text Label 2950 3050 0    50   ~ 0
+	3600 3150 3000 3150
+Text Label 3000 3150 0    50   ~ 0
 STOP_BUTTON
 Wire Wire Line
@@
 	5950 2950 5950 4150
 Wire Wire Line
-	5950 4150 2950 4150
+	5950 4150 3000 4150
 Wire Wire Line
-	2950 4150 2950 3050
+	3000 4150 3000 3150
+Wire Wire Line
+	3600 3050 2900 3050
+Wire Wire Line
+	2900 3050 2900 3250
+Wire Wire Line
+	2900 3250 2050 3250
+Wire Wire Line
+	2050 3250 2050 2750
+Wire Wire Line
+	2050 2750 1750 2750
+Text Label 2950 3050 0    50   ~ 0
+STOP_SWITCH
 $EndSCHEMATC

Commit message: -Lochraster Board -Errors fixed.
Connections:
- net labels removed: DECHO_BSWITCH, DTRIG_TSWITCH
Changed lines of the file:
@@
-	1    0    0    -1
-$EndComp
-$Comp
-L power:+5V #PWR01
-U 1 1 5C86D9D9
-P 9000 2800
-F 0 "#PWR01" H 9000 2650 50  0001 C CNN
-F 1 "+5V" H 9015 2973 50  0000 C CNN
-F 2 "" H 9000 2800 50  0001 C CNN
-F 3 "" H 9000 2800 50  0001 C CNN
-	1    9000 2800
 	1    0    0    -1
 $EndComp
@@
 	9400 4100 8350 4100
 Text Label 8350 3700 0    50   ~ 0
-DTRIG_TSWITCH
+TOP_SWITCH
 Text Label 2850 2050 0    50   ~ 0
 TOP_SWITCH
@@
 DCF77
 Text Label 8350 3800 0    50   ~ 0
-DECHO_BSWITCH
+BOTTOM_SWITCH
 Text Label 8350 3900 0    50   ~ 0
 STOP_SWITCH
@@
 Text Label 2950 3050 0    50   ~ 0
 STOP_SWITCH
+Text Label 8350 4200 0    50   ~ 0
+STOP_BUTTON
+Text Label 9000 2850 0    50   ~ 0
+3.3V
 $EndSCHEMATC
